Commit message: added lidar ignition systems but still lidar does not show up

File: icclab_summit_xl/urdf/sensors/hokuyo.urdf.xacro (robot description, xacro)
@@ -49,5 +49,5 @@
       <sensor type="ray" name="${prefix}_sensor">
         <pose>0 0 0 0 0 0</pose>
-        <visualize>false</visualize>
+        <topic>lidar</topic>
         <update_rate>30</update_rate>        <!-- 30 -->
         <ray>
@@ -71,5 +71,8 @@
           </noise>
         </ray>
-        <plugin name="${prefix}_controller" filename="libgazebo_ros_laser.so">
+        <always_on>1</always_on>
+        <visualize>true</visualize>
+        <plugin name="${prefix}_controller" filename="libignition-gazebo-sensors-system.so">
+          <render_engine>ogre2</render_engine>
           <topicName>${prefix_topic}</topicName>
           <frameName>/${prefix}_link</frameName>

File: icclab_summit_xl/urdf/sensors/hokuyo_utm30lx_no_frame_prefix.urdf.xacro (robot description, xacro)
@@ -39,13 +39,13 @@
 			<xacro:if value="${gpu}">
         <xacro:property name="ray_type" value="gpu_ray" />
-        <xacro:property name="plugin_lib" value="libgazebo_ros_gpu_laser.so" />
+        <xacro:property name="plugin_lib" value="libignition-gazebo-sensors-system.so" />
       </xacro:if>
       <xacro:unless value="${gpu}">
         <xacro:property name="ray_type" value="ray" />
-        <xacro:property name="plugin_lib" value="libgazebo_ros_ray_sensor.so" />
+        <xacro:property name="plugin_lib" value="libignition-gazebo-sensors-system.so" />
       </xacro:unless>
 			<sensor type="${ray_type}" name="${prefix}_sensor">
 				<pose>0 0 0 0 0 0</pose>
-				<visualize>false</visualize>
+        <topic>lidar</topic>
 				<update_rate>30</update_rate>
 				<ray>
@@ -69,4 +69,6 @@
 					</noise>
 				</ray>
+        <always_on>1</always_on>
+        <visualize>true</visualize>
 				<plugin name="${prefix}" filename="${plugin_lib}">
           <ros>
@@ -76,4 +78,5 @@
           <output_type>sensor_msgs/LaserScan</output_type>
 					<frame_name>${prefix}_link</frame_name>
+          <render_engine>ogre2</render_engine>
 				</plugin>
 			</sensor>
